Commit message: fix：robobus工程车外参

File: robobus_sensor_kit_description/urdf/sensor_kit.xacro (robot description, xacro)
@@ -19,4 +19,5 @@
     <link name="gnss" />
     <link name="os_sensor_top" />
+    <link name="os_sensor_ancillary" />
     <link name="os_sensor_fl" />
     <link name="os_sensor_fr" />
@@ -36,4 +37,15 @@
              ${calibration['sensor_kit_base_link']['os_sensor_top']['pitch']}
              ${calibration['sensor_kit_base_link']['os_sensor_top']['yaw']}" />
+    </joint>
+    <joint name="os_sensor_ancillary_joint" type="fixed">
+      <parent link="sensor_kit_base_link" />
+      <child link="os_sensor_ancillary" />
+      <origin
+        xyz="${calibration['sensor_kit_base_link']['os_sensor_ancillary']['x']}
+             ${calibration['sensor_kit_base_link']['os_sensor_ancillary']['y']}
+             ${calibration['sensor_kit_base_link']['os_sensor_ancillary']['z']}"
+        rpy="${calibration['sensor_kit_base_link']['os_sensor_ancillary']['roll']}
+             ${calibration['sensor_kit_base_link']['os_sensor_ancillary']['pitch']}
+             ${calibration['sensor_kit_base_link']['os_sensor_ancillary']['yaw']}" />
     </joint>
     <joint name="os_sensor_fl_joint" type="fixed">

Commit message: fix:ouster

File: robobus_sensor_kit_description/urdf/sensor_kit.xacro (robot description, xacro)
@@ -16,4 +16,5 @@
     <xacro:property name="calibration" value="${xacro.load_yaml('$(arg config_dir)/sensor_kit_calibration.yaml')}"/>
     <link name="traffic_light_left_camera" />
+    <link name="camera1" />
     <link name="zed" />
     <link name="gnss" />
@@ -105,4 +106,15 @@
              ${calibration['sensor_kit_base_link']['traffic_light_left_camera']['yaw']}" />
     </joint>
+    <joint name="camera1_joint" type="fixed">
+      <parent link="sensor_kit_base_link" />
+      <child link="camera1" />
+      <origin
+        xyz="${calibration['sensor_kit_base_link']['camera1']['x']}
+             ${calibration['sensor_kit_base_link']['camera1']['y']}
+             ${calibration['sensor_kit_base_link']['camera1']['z']}"
+        rpy="${calibration['sensor_kit_base_link']['camera1']['roll']}
+             ${calibration['sensor_kit_base_link']['camera1']['pitch']}
+             ${calibration['sensor_kit_base_link']['camera1']['yaw']}" />
+    </joint>
     <joint name="zed_joint" type="fixed">
       <parent link="sensor_kit_base_link" />
