Commit message: feat:muti ouster start launch file

File: robobus_sensor_kit_description/urdf/sensors.xacro (robot description, xacro)
@@ -6,6 +6,6 @@
   <link name="rs16" />
   <link name="rsbp" />
-  <link name="gnss" />
   <link name="os_sensor" />
+  <!-- robobus -->
   <link name="ultrasonic_0" />
   <link name="ultrasonic_1" />
@@ -17,4 +17,10 @@
   <link name="ultrasonic_7" />
   <link name="camera" />
+  <link name="gnss" />
+  <link name="os_sensor_top" />
+  <link name="os_sensor_fl" />
+  <link name="os_sensor_fr" />
+  <link name="os_sensor_rl" />
+  <link name="os_sensor_rr" />
   <xacro:arg name="config_dir" default="$(find robobus_sensor_kit_description)"/>
   <xacro:property name="calibration" value="${xacro.load_yaml('$(arg config_dir)/sensors_calibration.yaml')}"/>
@@ -39,9 +45,4 @@
     <child link="rs16" />
     <origin xyz="${calibration['base_link2rs16']['x']} ${calibration['base_link2rs16']['y']} ${calibration['base_link2rs16']['z']}" rpy="${calibration['base_link2rs16']['roll']} ${calibration['base_link2rs16']['pitch']} ${calibration['base_link2rs16']['yaw']}" />
-  </joint>
-  <joint name="baselink_gnss" type="fixed">
-    <parent link="base_link" />
-    <child link="gnss" />
-    <origin xyz="${calibration['base_link2gnss']['x']} ${calibration['base_link2gnss']['y']} ${calibration['base_link2gnss']['z']}" rpy="${calibration['base_link2gnss']['roll']} ${calibration['base_link2gnss']['pitch']} ${calibration['base_link2gnss']['yaw']}" />
   </joint>
   <joint name="baselink_ultrasonic_0" type="fixed">
@@ -85,8 +86,39 @@
     <origin xyz="${calibration['base_link2ultrasonic_7']['x']} ${calibration['base_link2ultrasonic_7']['y']} ${calibration['base_link2ultrasonic_7']['z']}" rpy="${calibration['base_link2ultrasonic_7']['roll']} ${calibration['base_link2ultrasonic_7']['pitch']} ${calibration['base_link2ultrasonic_7']['yaw']}" />
   </joint>
-  <joint name="rs16_camera" type="fixed">
-    <parent link="rs16" />
+  <!-- robobus -->
+  <joint name="baselink_gnss" type="fixed">
+    <parent link="base_link" />
+    <child link="gnss" />
+    <origin xyz="${calibration['base_link2gnss']['x']} ${calibration['base_link2gnss']['y']} ${calibration['base_link2gnss']['z']}" rpy="${calibration['base_link2gnss']['roll']} ${calibration['base_link2gnss']['pitch']} ${calibration['base_link2gnss']['yaw']}" />
+  </joint>
+  <joint name="top_os_camera" type="fixed">
+    <parent link="os_sensor_top" />
     <child link="camera" />
-    <origin xyz="${calibration['rs162camera']['x']} ${calibration['rs162camera']['y']} ${calibration['rs162camera']['z']}" rpy="${calibration['rs162camera']['roll']} ${calibration['rs162camera']['pitch']} ${calibration['rs162camera']['yaw']}" />
+    <origin xyz="${calibration['os_sensor_top2camera']['x']} ${calibration['os_sensor_top2camera']['y']} ${calibration['os_sensor_top2camera']['z']}" rpy="${calibration['os_sensor_top2camera']['roll']} ${calibration['os_sensor_top2camera']['pitch']} ${calibration['os_sensor_top2camera']['yaw']}" />
+  </joint>
+  <joint name="baselink_os_sensor_top" type="fixed">
+    <parent link="base_link" />
+    <child link="os_sensor_top" />
+    <origin xyz="${calibration['base_link2os_sensor_top']['x']} ${calibration['base_link2os_sensor_top']['y']} ${calibration['base_link2os_sensor_top']['z']}" rpy="${calibration['base_link2os_sensor_top']['roll']} ${calibration['base_link2os_sensor_top']['pitch']} ${calibration['base_link2os_sensor_top']['yaw']}" />
+  </joint>
+  <joint name="os_sensor_top_os_sensor_fl" type="fixed">
+    <parent link="os_sensor_top" />
+    <child link="os_sensor_fl" />
+    <origin xyz="${calibration['os_sensor_top2os_sensor_fl']['x']} ${calibration['os_sensor_top2os_sensor_fl']['y']} ${calibration['os_sensor_top2os_sensor_fl']['z']}" rpy="${calibration['os_sensor_top2os_sensor_fl']['roll']} ${calibration['os_sensor_top2os_sensor_fl']['pitch']} ${calibration['os_sensor_top2os_sensor_fl']['yaw']}" />
+  </joint>
+  <joint name="os_sensor_top_os_sensor_fr" type="fixed">
+    <parent link="os_sensor_top" />
+    <child link="os_sensor_fr" />
+    <origin xyz="${calibration['os_sensor_top2os_sensor_fr']['x']} ${calibration['os_sensor_top2os_sensor_fr']['y']} ${calibration['os_sensor_top2os_sensor_fr']['z']}" rpy="${calibration['os_sensor_top2os_sensor_fr']['roll']} ${calibration['os_sensor_top2os_sensor_fr']['pitch']} ${calibration['os_sensor_top2os_sensor_fr']['yaw']}" />
+  </joint>
+  <joint name="os_sensor_top_os_sensor_rl" type="fixed">
+    <parent link="os_sensor_top" />
+    <child link="os_sensor_rl" />
+    <origin xyz="${calibration['os_sensor_top2os_sensor_rl']['x']} ${calibration['os_sensor_top2os_sensor_rl']['y']} ${calibration['os_sensor_top2os_sensor_rl']['z']}" rpy="${calibration['os_sensor_top2os_sensor_rl']['roll']} ${calibration['os_sensor_top2os_sensor_rl']['pitch']} ${calibration['os_sensor_top2os_sensor_rl']['yaw']}" />
+  </joint>
+  <joint name="os_sensor_top_os_sensor_rr" type="fixed">
+    <parent link="os_sensor_top" />
+    <child link="os_sensor_rr" />
+    <origin xyz="${calibration['os_sensor_top2os_sensor_rr']['x']} ${calibration['os_sensor_top2os_sensor_rr']['y']} ${calibration['os_sensor_top2os_sensor_rr']['z']}" rpy="${calibration['os_sensor_top2os_sensor_rr']['roll']} ${calibration['os_sensor_top2os_sensor_rr']['pitch']} ${calibration['os_sensor_top2os_sensor_rr']['yaw']}" />
   </joint>
 </robot>

Commit message: feat: add gnss lidars

File: robobus_sensor_kit_description/urdf/sensors.xacro (robot description, xacro)
@@ -6,5 +6,5 @@
   <link name="rs16" />
   <link name="rsbp" />
-  <link name="os_sensor" />
+  <!-- <link name="os_sensor" /> -->
   <!-- robobus -->
   <link name="ultrasonic_0" />
@@ -26,9 +26,9 @@
   <xacro:property name="calibration" value="${xacro.load_yaml('$(arg config_dir)/sensors_calibration.yaml')}"/>
  <!-- embedded sensors -->
-  <joint name="baselink_os_sensor" type="fixed">
+  <!-- <joint name="baselink_os_sensor" type="fixed">
     <parent link="base_link" />
     <child link="os_sensor" />
     <origin xyz="${calibration['base_link2os_sensor']['x']} ${calibration['base_link2os_sensor']['y']} ${calibration['base_link2os_sensor']['z']}" rpy="${calibration['base_link2os_sensor']['roll']} ${calibration['base_link2os_sensor']['pitch']} ${calibration['base_link2os_sensor']['yaw']}" />
-  </joint>
+  </joint> -->
   <joint name="zed_baselink" type="fixed">
     <parent link="base_link" />

Commit message: fix:按照awsim_sensor_kit_launch的风格来编写

File: robobus_sensor_kit_description/urdf/sensors.xacro (robot description, xacro)
@@ -1,124 +1,98 @@
 <?xml version="1.0"?>
-<robot name="vehicle"
-  xmlns:xacro="http://ros.org/wiki/xacro">
-  <link name="zed_base_link" />
-  <!-- <link name="base_link" />  -->
-  <link name="rs16" />
-  <link name="rsbp" />
-  <!-- <link name="os_sensor" /> -->
-  <!-- robobus -->
-  <link name="ultrasonic_0" />
-  <link name="ultrasonic_1" />
-  <link name="ultrasonic_2" />
-  <link name="ultrasonic_3" />
-  <link name="ultrasonic_4" />
-  <link name="ultrasonic_5" />
-  <link name="ultrasonic_6" />
-  <link name="ultrasonic_7" />
-  <link name="camera" />
-  <link name="gnss" />
-  <link name="os_sensor_top" />
-  <link name="os_sensor_fl" />
-  <link name="os_sensor_fr" />
-  <link name="os_sensor_rl" />
-  <link name="os_sensor_rr" />
-  <xacro:arg name="config_dir" default="$(find robobus_sensor_kit_description)"/>
+<robot name="vehicle" xmlns:xacro="http://ros.org/wiki/xacro">
+  <xacro:arg name="config_dir" default="$(find robobus_sensor_kit_description)/config"/>
   <xacro:property name="calibration" value="${xacro.load_yaml('$(arg config_dir)/sensors_calibration.yaml')}"/>
- <!-- embedded sensors -->
-  <!-- <joint name="baselink_os_sensor" type="fixed">
-    <parent link="base_link" />
-    <child link="os_sensor" />
-    <origin xyz="${calibration['base_link2os_sensor']['x']} ${calibration['base_link2os_sensor']['y']} ${calibration['base_link2os_sensor']['z']}" rpy="${calibration['base_link2os_sensor']['roll']} ${calibration['base_link2os_sensor']['pitch']} ${calibration['base_link2os_sensor']['yaw']}" />
-  </joint> -->
-  <joint name="zed_baselink" type="fixed">
-    <parent link="base_link" />
-    <child link="zed_base_link" />
-    <origin xyz="${calibration['base_link2zed']['x']} ${calibration['base_link2zed']['y']} ${calibration['base_link2zed']['z']}" rpy="${calibration['base_link2zed']['roll']} ${calibration['base_link2zed']['pitch']} ${calibration['base_link2zed']['yaw']}" />
-    </joint>
-  <joint name="baselink_rsbp" type="fixed">
-    <parent link="base_link" />
-    <child link="rsbp" />
-    <origin xyz="${calibration['base_link2rsbp']['x']} ${calibration['base_link2rsbp']['y']} ${calibration['base_link2rsbp']['z']}" rpy="${calibration['base_link2rsbp']['roll']} ${calibration['base_link2rsbp']['pitch']} ${calibration['base_link2rsbp']['yaw']}" />
-  </joint>
-  <joint name="baselink_rs16" type="fixed">
-    <parent link="base_link" />
-    <child link="rs16" />
-    <origin xyz="${calibration['base_link2rs16']['x']} ${calibration['base_link2rs16']['y']} ${calibration['base_link2rs16']['z']}" rpy="${calibration['base_link2rs16']['roll']} ${calibration['base_link2rs16']['pitch']} ${calibration['base_link2rs16']['yaw']}" />
-  </joint>
-  <joint name="baselink_ultrasonic_0" type="fixed">
-    <parent link="base_link" />
-    <child link="ultrasonic_0" />
-    <origin xyz="${calibration['base_link2ultrasonic_0']['x']} ${calibration['base_link2ultrasonic_0']['y']} ${calibration['base_link2ultrasonic_0']['z']}" rpy="${calibration['base_link2ultrasonic_0']['roll']} ${calibration['base_link2ultrasonic_0']['pitch']} ${calibration['base_link2ultrasonic_0']['yaw']}" />
-  </joint>
-  <joint name="baselink_ultrasonic_1" type="fixed">
-    <parent link="base_link" />
-    <child link="ultrasonic_1" />
-    <origin xyz="${calibration['base_link2ultrasonic_1']['x']} ${calibration['base_link2ultrasonic_1']['y']} ${calibration['base_link2ultrasonic_1']['z']}" rpy="${calibration['base_link2ultrasonic_1']['roll']} ${calibration['base_link2ultrasonic_1']['pitch']} ${calibration['base_link2ultrasonic_1']['yaw']}" />
-  </joint>
-  <joint name="baselink_ultrasonic_2" type="fixed">
-    <parent link="base_link" />
-    <child link="ultrasonic_2" />
-    <origin xyz="${calibration['base_link2ultrasonic_2']['x']} ${calibration['base_link2ultrasonic_2']['y']} ${calibration['base_link2ultrasonic_2']['z']}" rpy="${calibration['base_link2ultrasonic_2']['roll']} ${calibration['base_link2ultrasonic_2']['pitch']} ${calibration['base_link2ultrasonic_2']['yaw']}" />
-  </joint>
-  <joint name="baselink_ultrasonic_3" type="fixed">
-    <parent link="base_link" />
-    <child link="ultrasonic_3" />
-    <origin xyz="${calibration['base_link2ultrasonic_3']['x']} ${calibration['base_link2ultrasonic_3']['y']} ${calibration['base_link2ultrasonic_3']['z']}" rpy="${calibration['base_link2ultrasonic_3']['roll']} ${calibration['base_link2ultrasonic_3']['pitch']} ${calibration['base_link2ultrasonic_3']['yaw']}" />
-  </joint>
-  <joint name="baselink_ultrasonic_4" type="fixed">
-    <parent link="base_link" />
-    <child link="ultrasonic_4" />
-    <origin xyz="${calibration['base_link2ultrasonic_4']['x']} ${calibration['base_link2ultrasonic_4']['y']} ${calibration['base_link2ultrasonic_4']['z']}" rpy="${calibration['base_link2ultrasonic_4']['roll']} ${calibration['base_link2ultrasonic_4']['pitch']} ${calibration['base_link2ultrasonic_4']['yaw']}" />
-  </joint>
-  <joint name="baselink_ultrasonic_5" type="fixed">
-    <parent link="base_link" />
-    <child link="ultrasonic_5" />
-    <origin xyz="${calibration['base_link2ultrasonic_5']['x']} ${calibration['base_link2ultrasonic_5']['y']} ${calibration['base_link2ultrasonic_5']['z']}" rpy="${calibration['base_link2ultrasonic_5']['roll']} ${calibration['base_link2ultrasonic_5']['pitch']} ${calibration['base_link2ultrasonic_5']['yaw']}" />
-  </joint>
-  <joint name="baselink_ultrasonic_6" type="fixed">
-    <parent link="base_link" />
-    <child link="ultrasonic_6" />
-    <origin xyz="${calibration['base_link2ultrasonic_6']['x']} ${calibration['base_link2ultrasonic_6']['y']} ${calibration['base_link2ultrasonic_6']['z']}" rpy="${calibration['base_link2ultrasonic_6']['roll']} ${calibration['base_link2ultrasonic_6']['pitch']} ${calibration['base_link2ultrasonic_6']['yaw']}" />
-  </joint>
-  <joint name="baselink_ultrasonic_7" type="fixed">
-    <parent link="base_link" />
-    <child link="ultrasonic_7" />
-    <origin xyz="${calibration['base_link2ultrasonic_7']['x']} ${calibration['base_link2ultrasonic_7']['y']} ${calibration['base_link2ultrasonic_7']['z']}" rpy="${calibration['base_link2ultrasonic_7']['roll']} ${calibration['base_link2ultrasonic_7']['pitch']} ${calibration['base_link2ultrasonic_7']['yaw']}" />
-  </joint>
-  <!-- robobus -->
-  <joint name="baselink_gnss" type="fixed">
-    <parent link="base_link" />
-    <child link="gnss" />
-    <origin xyz="${calibration['base_link2gnss']['x']} ${calibration['base_link2gnss']['y']} ${calibration['base_link2gnss']['z']}" rpy="${calibration['base_link2gnss']['roll']} ${calibration['base_link2gnss']['pitch']} ${calibration['base_link2gnss']['yaw']}" />
-  </joint>
-  <joint name="top_os_camera" type="fixed">
-    <parent link="os_sensor_top" />
-    <child link="camera" />
-    <origin xyz="${calibration['os_sensor_top2camera']['x']} ${calibration['os_sensor_top2camera']['y']} ${calibration['os_sensor_top2camera']['z']}" rpy="${calibration['os_sensor_top2camera']['roll']} ${calibration['os_sensor_top2camera']['pitch']} ${calibration['os_sensor_top2camera']['yaw']}" />
-  </joint>
-  <joint name="baselink_os_sensor_top" type="fixed">
-    <parent link="base_link" />
-    <child link="os_sensor_top" />
-    <origin xyz="${calibration['base_link2os_sensor_top']['x']} ${calibration['base_link2os_sensor_top']['y']} ${calibration['base_link2os_sensor_top']['z']}" rpy="${calibration['base_link2os_sensor_top']['roll']} ${calibration['base_link2os_sensor_top']['pitch']} ${calibration['base_link2os_sensor_top']['yaw']}" />
-  </joint>
-  <joint name="os_sensor_top_os_sensor_fl" type="fixed">
-    <parent link="os_sensor_top" />
-    <child link="os_sensor_fl" />
-    <origin xyz="${calibration['os_sensor_top2os_sensor_fl']['x']} ${calibration['os_sensor_top2os_sensor_fl']['y']} ${calibration['os_sensor_top2os_sensor_fl']['z']}" rpy="${calibration['os_sensor_top2os_sensor_fl']['roll']} ${calibration['os_sensor_top2os_sensor_fl']['pitch']} ${calibration['os_sensor_top2os_sensor_fl']['yaw']}" />
-  </joint>
-  <joint name="os_sensor_top_os_sensor_fr" type="fixed">
-    <parent link="os_sensor_top" />
-    <child link="os_sensor_fr" />
-    <origin xyz="${calibration['os_sensor_top2os_sensor_fr']['x']} ${calibration['os_sensor_top2os_sensor_fr']['y']} ${calibration['os_sensor_top2os_sensor_fr']['z']}" rpy="${calibration['os_sensor_top2os_sensor_fr']['roll']} ${calibration['os_sensor_top2os_sensor_fr']['pitch']} ${calibration['os_sensor_top2os_sensor_fr']['yaw']}" />
-  </joint>
-  <joint name="os_sensor_top_os_sensor_rl" type="fixed">
-    <parent link="os_sensor_top" />
-    <child link="os_sensor_rl" />
-    <origin xyz="${calibration['os_sensor_top2os_sensor_rl']['x']} ${calibration['os_sensor_top2os_sensor_rl']['y']} ${calibration['os_sensor_top2os_sensor_rl']['z']}" rpy="${calibration['os_sensor_top2os_sensor_rl']['roll']} ${calibration['os_sensor_top2os_sensor_rl']['pitch']} ${calibration['os_sensor_top2os_sensor_rl']['yaw']}" />
-  </joint>
-  <joint name="os_sensor_top_os_sensor_rr" type="fixed">
-    <parent link="os_sensor_top" />
-    <child link="os_sensor_rr" />
-    <origin xyz="${calibration['os_sensor_top2os_sensor_rr']['x']} ${calibration['os_sensor_top2os_sensor_rr']['y']} ${calibration['os_sensor_top2os_sensor_rr']['z']}" rpy="${calibration['os_sensor_top2os_sensor_rr']['roll']} ${calibration['os_sensor_top2os_sensor_rr']['pitch']} ${calibration['os_sensor_top2os_sensor_rr']['yaw']}" />
-  </joint>
+  <!-- sensor kit -->
+  <xacro:include filename="sensor_kit.xacro"/>
+  <xacro:sensor_kit_macro parent="base_link">
+    <origin
+      xyz="${calibration['base_link']['sensor_kit_base_link']['x']}
+           ${calibration['base_link']['sensor_kit_base_link']['y']}
+           ${calibration['base_link']['sensor_kit_base_link']['z']}"
+      rpy="${calibration['base_link']['sensor_kit_base_link']['roll']}
+           ${calibration['base_link']['sensor_kit_base_link']['pitch']}
+           ${calibration['base_link']['sensor_kit_base_link']['yaw']}"
+    />
+  </xacro:sensor_kit_macro>
+  <!-- ultrasonic -->
+  <xacro:ultrasonic_0 >
+    <origin
+      xyz="${calibration['base_link']['ultrasonic_0']['x']}
+           ${calibration['base_link']['ultrasonic_0']['y']}
+           ${calibration['base_link']['ultrasonic_0']['z']}"
+      rpy="${calibration['base_link']['ultrasonic_0']['roll']}
+           ${calibration['base_link']['ultrasonic_0']['pitch']}
+           ${calibration['base_link']['ultrasonic_0']['yaw']}"
+    />
+  </xacro:ultrasonic_0>
+  <xacro:ultrasonic_1 >
+    <origin
+      xyz="${calibration['base_link']['ultrasonic_1']['x']}
+           ${calibration['base_link']['ultrasonic_1']['y']}
+           ${calibration['base_link']['ultrasonic_1']['z']}"
+      rpy="${calibration['base_link']['ultrasonic_1']['roll']}
+           ${calibration['base_link']['ultrasonic_1']['pitch']}
+           ${calibration['base_link']['ultrasonic_1']['yaw']}"
+    />
+  </xacro:ultrasonic_1>
+  <xacro:ultrasonic_2 >
+    <origin
+      xyz="${calibration['base_link']['ultrasonic_2']['x']}
+           ${calibration['base_link']['ultrasonic_2']['y']}
+           ${calibration['base_link']['ultrasonic_2']['z']}"
+      rpy="${calibration['base_link']['ultrasonic_2']['roll']}
+           ${calibration['base_link']['ultrasonic_2']['pitch']}
+           ${calibration['base_link']['ultrasonic_2']['yaw']}"
+    />
+  </xacro:ultrasonic_2>
+  <xacro:ultrasonic_3 >
+    <origin
+      xyz="${calibration['base_link']['ultrasonic_3']['x']}
+           ${calibration['base_link']['ultrasonic_3']['y']}
+           ${calibration['base_link']['ultrasonic_3']['z']}"
+      rpy="${calibration['base_link']['ultrasonic_3']['roll']}
+           ${calibration['base_link']['ultrasonic_3']['pitch']}
+           ${calibration['base_link']['ultrasonic_3']['yaw']}"
+    />
+  </xacro:ultrasonic_3>
+  <xacro:ultrasonic_4 >
+    <origin
+      xyz="${calibration['base_link']['ultrasonic_4']['x']}
+           ${calibration['base_link']['ultrasonic_4']['y']}
+           ${calibration['base_link']['ultrasonic_4']['z']}"
+      rpy="${calibration['base_link']['ultrasonic_4']['roll']}
+           ${calibration['base_link']['ultrasonic_4']['pitch']}
+           ${calibration['base_link']['ultrasonic_4']['yaw']}"
+    />
+  </xacro:ultrasonic_4>
+  <xacro:ultrasonic_5 >
+    <origin
+      xyz="${calibration['base_link']['ultrasonic_5']['x']}
+           ${calibration['base_link']['ultrasonic_5']['y']}
+           ${calibration['base_link']['ultrasonic_5']['z']}"
+      rpy="${calibration['base_link']['ultrasonic_5']['roll']}
+           ${calibration['base_link']['ultrasonic_5']['pitch']}
+           ${calibration['base_link']['ultrasonic_5']['yaw']}"
+    />
+  </xacro:ultrasonic_5>
+  <xacro:ultrasonic_6 >
+    <origin
+      xyz="${calibration['base_link']['ultrasonic_6']['x']}
+           ${calibration['base_link']['ultrasonic_6']['y']}
+           ${calibration['base_link']['ultrasonic_6']['z']}"
+      rpy="${calibration['base_link']['ultrasonic_6']['roll']}
+           ${calibration['base_link']['ultrasonic_6']['pitch']}
+           ${calibration['base_link']['ultrasonic_6']['yaw']}"
+    />
+  </xacro:ultrasonic_6>
+  <xacro:ultrasonic_7 >
+    <origin
+      xyz="${calibration['base_link']['ultrasonic_7']['x']}
+           ${calibration['base_link']['ultrasonic_7']['y']}
+           ${calibration['base_link']['ultrasonic_7']['z']}"
+      rpy="${calibration['base_link']['ultrasonic_7']['roll']}
+           ${calibration['base_link']['ultrasonic_7']['pitch']}
+           ${calibration['base_link']['ultrasonic_7']['yaw']}"
+    />
+  </xacro:ultrasonic_7>
 </robot>
