Commit message: fix: 方便标定方式编写

File: robobus_sensor_kit_description/urdf/sensors.xacro (robot description, xacro)
@@ -3,96 +3,93 @@
   <xacro:arg name="config_dir" default="$(find robobus_sensor_kit_description)/config"/>
   <xacro:property name="calibration" value="${xacro.load_yaml('$(arg config_dir)/sensors_calibration.yaml')}"/>
-  <!-- sensor kit -->
-  <xacro:include filename="sensor_kit.xacro"/>
-  <xacro:sensor_kit_macro parent="base_link">
+  <xacro:include filename="sensors_secondary.xacro"/>
+  <!-- sensor kit link -->
+  <link name="traffic_light_left_camera" />
+  <link name="camera1" />
+  <link name="os_lidar_fl" />
+  <link name="os_lidar_fr" />
+  <link name="os_lidar_rl" />
+  <link name="os_lidar_rr" />
+  <link name="gnss" />
+  <!-- sensor kit joint -->
+  <!-- camera -->
+  <joint name="camera1_joint" type="fixed">
+    <parent link="rs16" />
+    <child link="camera1" />
     <origin
-      xyz="${calibration['base_link']['sensor_kit_base_link']['x']}
-           ${calibration['base_link']['sensor_kit_base_link']['y']}
-           ${calibration['base_link']['sensor_kit_base_link']['z']}"
-      rpy="${calibration['base_link']['sensor_kit_base_link']['roll']}
-           ${calibration['base_link']['sensor_kit_base_link']['pitch']}
-           ${calibration['base_link']['sensor_kit_base_link']['yaw']}"
-    />
-  </xacro:sensor_kit_macro>
-  <!-- ultrasonic -->
-  <xacro:ultrasonic_0 >
+      xyz="${calibration['rs16']['camera1']['x']}
+            ${calibration['rs16']['camera1']['y']}
+            ${calibration['rs16']['camera1']['z']}"
+      rpy="${calibration['rs16']['camera1']['roll']}
+            ${calibration['rs16']['camera1']['pitch']}
+            ${calibration['rs16']['camera1']['yaw']}" />
+  </joint>
+  <joint name="traffic_light_left_camera_joint" type="fixed">
+    <parent link="rs16" />
+    <child link="traffic_light_left_camera" />
     <origin
-      xyz="${calibration['base_link']['ultrasonic_0']['x']}
-           ${calibration['base_link']['ultrasonic_0']['y']}
-           ${calibration['base_link']['ultrasonic_0']['z']}"
-      rpy="${calibration['base_link']['ultrasonic_0']['roll']}
-           ${calibration['base_link']['ultrasonic_0']['pitch']}
-           ${calibration['base_link']['ultrasonic_0']['yaw']}"
-    />
-  </xacro:ultrasonic_0>
-  <xacro:ultrasonic_1 >
+      xyz="${calibration['rs16']['traffic_light_left_camera']['x']}
+            ${calibration['rs16']['traffic_light_left_camera']['y']}
+            ${calibration['rs16']['traffic_light_left_camera']['z']}"
+      rpy="${calibration['rs16']['traffic_light_left_camera']['roll']}
+            ${calibration['rs16']['traffic_light_left_camera']['pitch']}
+            ${calibration['rs16']['traffic_light_left_camera']['yaw']}" />
+  </joint>
+  <!-- lidar  -->
+  <joint name="os_lidar_fl_joint" type="fixed">
+    <parent link="rs16" />
+    <child link="os_lidar_fl" />
     <origin
-      xyz="${calibration['base_link']['ultrasonic_1']['x']}
-           ${calibration['base_link']['ultrasonic_1']['y']}
-           ${calibration['base_link']['ultrasonic_1']['z']}"
-      rpy="${calibration['base_link']['ultrasonic_1']['roll']}
-           ${calibration['base_link']['ultrasonic_1']['pitch']}
-           ${calibration['base_link']['ultrasonic_1']['yaw']}"
-    />
-  </xacro:ultrasonic_1>
-  <xacro:ultrasonic_2 >
+      xyz="${calibration['rs16']['os_lidar_fl']['x']}
+            ${calibration['rs16']['os_lidar_fl']['y']}
+            ${calibration['rs16']['os_lidar_fl']['z']}"
+      rpy="${calibration['rs16']['os_lidar_fl']['roll']}
+            ${calibration['rs16']['os_lidar_fl']['pitch']}
+            ${calibration['rs16']['os_lidar_fl']['yaw']}" />
+  </joint>
+  <joint name="os_lidar_fr_joint" type="fixed">
+    <parent link="rs16" />
+    <child link="os_lidar_fr" />
     <origin
-      xyz="${calibration['base_link']['ultrasonic_2']['x']}
-           ${calibration['base_link']['ultrasonic_2']['y']}
-           ${calibration['base_link']['ultrasonic_2']['z']}"
-      rpy="${calibration['base_link']['ultrasonic_2']['roll']}
-           ${calibration['base_link']['ultrasonic_2']['pitch']}
-           ${calibration['base_link']['ultrasonic_2']['yaw']}"
-    />
-  </xacro:ultrasonic_2>
-  <xacro:ultrasonic_3 >
+      xyz="${calibration['rs16']['os_lidar_fr']['x']}
+            ${calibration['rs16']['os_lidar_fr']['y']}
+            ${calibration['rs16']['os_lidar_fr']['z']}"
+      rpy="${calibration['rs16']['os_lidar_fr']['roll']}
+            ${calibration['rs16']['os_lidar_fr']['pitch']}
+            ${calibration['rs16']['os_lidar_fr']['yaw']}" />
+  </joint>
+   <joint name="os_lidar_rl_joint" type="fixed">
+    <parent link="rs16" />
+    <child link="os_lidar_rl" />
     <origin
-      xyz="${calibration['base_link']['ultrasonic_3']['x']}
-           ${calibration['base_link']['ultrasonic_3']['y']}
-           ${calibration['base_link']['ultrasonic_3']['z']}"
-      rpy="${calibration['base_link']['ultrasonic_3']['roll']}
-           ${calibration['base_link']['ultrasonic_3']['pitch']}
-           ${calibration['base_link']['ultrasonic_3']['yaw']}"
-    />
-  </xacro:ultrasonic_3>
-  <xacro:ultrasonic_4 >
+      xyz="${calibration['rs16']['os_lidar_rl']['x']}
+            ${calibration['rs16']['os_lidar_rl']['y']}
+            ${calibration['rs16']['os_lidar_rl']['z']}"
+      rpy="${calibration['rs16']['os_lidar_rl']['roll']}
+            ${calibration['rs16']['os_lidar_rl']['pitch']}
+            ${calibration['rs16']['os_lidar_rl']['yaw']}" />
+  </joint>
+   <joint name="os_lidar_rr_joint" type="fixed">
+    <parent link="rs16" />
+    <child link="os_lidar_rr" />
     <origin
-      xyz="${calibration['base_link']['ultrasonic_4']['x']}
-           ${calibration['base_link']['ultrasonic_4']['y']}
-           ${calibration['base_link']['ultrasonic_4']['z']}"
-      rpy="${calibration['base_link']['ultrasonic_4']['roll']}
-           ${calibration['base_link']['ultrasonic_4']['pitch']}
-           ${calibration['base_link']['ultrasonic_4']['yaw']}"
-    />
-  </xacro:ultrasonic_4>
-  <xacro:ultrasonic_5 >
+      xyz="${calibration['rs16']['os_lidar_rr']['x']}
+            ${calibration['rs16']['os_lidar_rr']['y']}
+            ${calibration['rs16']['os_lidar_rr']['z']}"
+      rpy="${calibration['rs16']['os_lidar_rr']['roll']}
+            ${calibration['rs16']['os_lidar_rr']['pitch']}
+            ${calibration['rs16']['os_lidar_rr']['yaw']}" />
+  </joint>
+<!-- combined navigation -->
+  <joint name="gnss_joint" type="fixed">
+    <parent link="rs16" />
+    <child link="gnss" />
     <origin
-      xyz="${calibration['base_link']['ultrasonic_5']['x']}
-           ${calibration['base_link']['ultrasonic_5']['y']}
-           ${calibration['base_link']['ultrasonic_5']['z']}"
-      rpy="${calibration['base_link']['ultrasonic_5']['roll']}
-           ${calibration['base_link']['ultrasonic_5']['pitch']}
-           ${calibration['base_link']['ultrasonic_5']['yaw']}"
-    />
-  </xacro:ultrasonic_5>
-  <xacro:ultrasonic_6 >
-    <origin
-      xyz="${calibration['base_link']['ultrasonic_6']['x']}
-           ${calibration['base_link']['ultrasonic_6']['y']}
-           ${calibration['base_link']['ultrasonic_6']['z']}"
-      rpy="${calibration['base_link']['ultrasonic_6']['roll']}
-           ${calibration['base_link']['ultrasonic_6']['pitch']}
-           ${calibration['base_link']['ultrasonic_6']['yaw']}"
-    />
-  </xacro:ultrasonic_6>
-  <xacro:ultrasonic_7 >
-    <origin
-      xyz="${calibration['base_link']['ultrasonic_7']['x']}
-           ${calibration['base_link']['ultrasonic_7']['y']}
-           ${calibration['base_link']['ultrasonic_7']['z']}"
-      rpy="${calibration['base_link']['ultrasonic_7']['roll']}
-           ${calibration['base_link']['ultrasonic_7']['pitch']}
-           ${calibration['base_link']['ultrasonic_7']['yaw']}"
-    />
-  </xacro:ultrasonic_7>
+      xyz="${calibration['rs16']['gnss']['x']}
+            ${calibration['rs16']['gnss']['y']}
+            ${calibration['rs16']['gnss']['z']}"
+      rpy="${calibration['rs16']['gnss']['roll']}
+            ${calibration['rs16']['gnss']['pitch']}
+            ${calibration['rs16']['gnss']['yaw']}" />
+  </joint>
 </robot>

Commit message: feat:传感器描述文件重构

File: robobus_sensor_kit_description/urdf/sensors.xacro (robot description, xacro)
@@ -7,4 +7,5 @@
   <link name="traffic_light_left_camera" />
   <link name="camera1" />
+  <link name="os_lidar_ancillary" />
   <link name="os_lidar_fl" />
   <link name="os_lidar_fr" />
@@ -13,26 +14,37 @@
   <link name="gnss" />
   <!-- sensor kit joint -->
+  <joint name="os_lidar_ancillary_joint" type="fixed">
+    <parent link="rs16" />
+    <child link="os_lidar_ancillary" />
+    <origin
+      xyz="${calibration['rs16']['os_lidar_ancillary']['x']}
+            ${calibration['rs16']['os_lidar_ancillary']['y']}
+            ${calibration['rs16']['os_lidar_ancillary']['z']}"
+      rpy="${calibration['rs16']['os_lidar_ancillary']['roll']}
+            ${calibration['rs16']['os_lidar_ancillary']['pitch']}
+            ${calibration['rs16']['os_lidar_ancillary']['yaw']}" />
+  </joint>
   <!-- camera -->
   <joint name="camera1_joint" type="fixed">
-    <parent link="rs16" />
+    <parent link="os_lidar_ancillary" />
     <child link="camera1" />
     <origin
-      xyz="${calibration['rs16']['camera1']['x']}
-            ${calibration['rs16']['camera1']['y']}
-            ${calibration['rs16']['camera1']['z']}"
-      rpy="${calibration['rs16']['camera1']['roll']}
-            ${calibration['rs16']['camera1']['pitch']}
-            ${calibration['rs16']['camera1']['yaw']}" />
+      xyz="${calibration['os_lidar_ancillary']['camera1']['x']}
+            ${calibration['os_lidar_ancillary']['camera1']['y']}
+            ${calibration['os_lidar_ancillary']['camera1']['z']}"
+      rpy="${calibration['os_lidar_ancillary']['camera1']['roll']}
+            ${calibration['os_lidar_ancillary']['camera1']['pitch']}
+            ${calibration['os_lidar_ancillary']['camera1']['yaw']}" />
   </joint>
   <joint name="traffic_light_left_camera_joint" type="fixed">
-    <parent link="rs16" />
+    <parent link="os_lidar_ancillary" />
     <child link="traffic_light_left_camera" />
     <origin
-      xyz="${calibration['rs16']['traffic_light_left_camera']['x']}
-            ${calibration['rs16']['traffic_light_left_camera']['y']}
-            ${calibration['rs16']['traffic_light_left_camera']['z']}"
-      rpy="${calibration['rs16']['traffic_light_left_camera']['roll']}
-            ${calibration['rs16']['traffic_light_left_camera']['pitch']}
-            ${calibration['rs16']['traffic_light_left_camera']['yaw']}" />
+      xyz="${calibration['os_lidar_ancillary']['traffic_light_left_camera']['x']}
+            ${calibration['os_lidar_ancillary']['traffic_light_left_camera']['y']}
+            ${calibration['os_lidar_ancillary']['traffic_light_left_camera']['z']}"
+      rpy="${calibration['os_lidar_ancillary']['traffic_light_left_camera']['roll']}
+            ${calibration['os_lidar_ancillary']['traffic_light_left_camera']['pitch']}
+            ${calibration['os_lidar_ancillary']['traffic_light_left_camera']['yaw']}" />
   </joint>
   <!-- lidar  -->

File: robobus_sensor_kit_description/urdf/sensors_secondary.xacro (robot description, xacro)
@@ -5,5 +5,4 @@
   <!-- sensor secondary link -->
   <link name="rs16" />
-  <link name="os_lidar_ancillary" />
   <link name="front_radar" />
   <link name="rear_radar" />
@@ -32,15 +31,4 @@
             ${secondary_calibration['base_link']['rs16']['pitch']}
             ${secondary_calibration['base_link']['rs16']['yaw']}" />
-  </joint>
-  <joint name="os_lidar_ancillary_joint" type="fixed">
-    <parent link="base_link" />
-    <child link="os_lidar_ancillary" />
-    <origin
-      xyz="${secondary_calibration['base_link']['os_lidar_ancillary']['x']}
-            ${secondary_calibration['base_link']['os_lidar_ancillary']['y']}
-            ${secondary_calibration['base_link']['os_lidar_ancillary']['z']}"
-      rpy="${secondary_calibration['base_link']['os_lidar_ancillary']['roll']}
-            ${secondary_calibration['base_link']['os_lidar_ancillary']['pitch']}
-            ${secondary_calibration['base_link']['os_lidar_ancillary']['yaw']}" />
   </joint>
   <!-- millimeter wave -->

Commit message: fix:

File: robobus_sensor_kit_description/urdf/sensors.xacro (robot description, xacro)
@@ -5,6 +5,6 @@
   <xacro:include filename="sensors_secondary.xacro"/>
   <!-- sensor kit link -->
-  <link name="traffic_light_left_camera" />
-  <link name="camera1" />
+  <link name="camera_top" />
+  <link name="camera_front" />
   <link name="os_lidar_ancillary" />
   <link name="os_lidar_fl" />
@@ -26,25 +26,25 @@
   </joint>
   <!-- camera -->
-  <joint name="camera1_joint" type="fixed">
+  <joint name="camera_front_joint" type="fixed">
     <parent link="os_lidar_ancillary" />
-    <child link="camera1" />
+    <child link="camera_front" />
     <origin
-      xyz="${calibration['os_lidar_ancillary']['camera1']['x']}
-            ${calibration['os_lidar_ancillary']['camera1']['y']}
-            ${calibration['os_lidar_ancillary']['camera1']['z']}"
-      rpy="${calibration['os_lidar_ancillary']['camera1']['roll']}
-            ${calibration['os_lidar_ancillary']['camera1']['pitch']}
-            ${calibration['os_lidar_ancillary']['camera1']['yaw']}" />
+      xyz="${calibration['os_lidar_ancillary']['camera_front']['x']}
+            ${calibration['os_lidar_ancillary']['camera_front']['y']}
+            ${calibration['os_lidar_ancillary']['camera_front']['z']}"
+      rpy="${calibration['os_lidar_ancillary']['camera_front']['roll']}
+            ${calibration['os_lidar_ancillary']['camera_front']['pitch']}
+            ${calibration['os_lidar_ancillary']['camera_front']['yaw']}" />
   </joint>
-  <joint name="traffic_light_left_camera_joint" type="fixed">
+  <joint name="camera_top_joint" type="fixed">
     <parent link="os_lidar_ancillary" />
-    <child link="traffic_light_left_camera" />
+    <child link="camera_top" />
     <origin
-      xyz="${calibration['os_lidar_ancillary']['traffic_light_left_camera']['x']}
-            ${calibration['os_lidar_ancillary']['traffic_light_left_camera']['y']}
-            ${calibration['os_lidar_ancillary']['traffic_light_left_camera']['z']}"
-      rpy="${calibration['os_lidar_ancillary']['traffic_light_left_camera']['roll']}
-            ${calibration['os_lidar_ancillary']['traffic_light_left_camera']['pitch']}
-            ${calibration['os_lidar_ancillary']['traffic_light_left_camera']['yaw']}" />
+      xyz="${calibration['os_lidar_ancillary']['camera_top']['x']}
+            ${calibration['os_lidar_ancillary']['camera_top']['y']}
+            ${calibration['os_lidar_ancillary']['camera_top']['z']}"
+      rpy="${calibration['os_lidar_ancillary']['camera_top']['roll']}
+            ${calibration['os_lidar_ancillary']['camera_top']['pitch']}
+            ${calibration['os_lidar_ancillary']['camera_top']['yaw']}" />
   </joint>
   <!-- lidar  -->

Commit message: fix: 修改顶部lidar frame

File: robobus_sensor_kit_description/urdf/sensors.xacro (robot description, xacro)
@@ -15,13 +15,13 @@
   <!-- sensor kit joint -->
   <joint name="os_lidar_ancillary_joint" type="fixed">
-    <parent link="rs16" />
+    <parent link="sensor_top" />
     <child link="os_lidar_ancillary" />
     <origin
-      xyz="${calibration['rs16']['os_lidar_ancillary']['x']}
-            ${calibration['rs16']['os_lidar_ancillary']['y']}
-            ${calibration['rs16']['os_lidar_ancillary']['z']}"
-      rpy="${calibration['rs16']['os_lidar_ancillary']['roll']}
-            ${calibration['rs16']['os_lidar_ancillary']['pitch']}
-            ${calibration['rs16']['os_lidar_ancillary']['yaw']}" />
+      xyz="${calibration['sensor_top']['os_lidar_ancillary']['x']}
+            ${calibration['sensor_top']['os_lidar_ancillary']['y']}
+            ${calibration['sensor_top']['os_lidar_ancillary']['z']}"
+      rpy="${calibration['sensor_top']['os_lidar_ancillary']['roll']}
+            ${calibration['sensor_top']['os_lidar_ancillary']['pitch']}
+            ${calibration['sensor_top']['os_lidar_ancillary']['yaw']}" />
   </joint>
   <!-- camera -->
@@ -50,58 +50,58 @@
   <!-- lidar  -->
   <joint name="os_lidar_fl_joint" type="fixed">
-    <parent link="rs16" />
+    <parent link="sensor_top" />
     <child link="os_lidar_fl" />
     <origin
-      xyz="${calibration['rs16']['os_lidar_fl']['x']}
-            ${calibration['rs16']['os_lidar_fl']['y']}
-            ${calibration['rs16']['os_lidar_fl']['z']}"
-      rpy="${calibration['rs16']['os_lidar_fl']['roll']}
-            ${calibration['rs16']['os_lidar_fl']['pitch']}
-            ${calibration['rs16']['os_lidar_fl']['yaw']}" />
+      xyz="${calibration['sensor_top']['os_lidar_fl']['x']}
+            ${calibration['sensor_top']['os_lidar_fl']['y']}
+            ${calibration['sensor_top']['os_lidar_fl']['z']}"
+      rpy="${calibration['sensor_top']['os_lidar_fl']['roll']}
+            ${calibration['sensor_top']['os_lidar_fl']['pitch']}
+            ${calibration['sensor_top']['os_lidar_fl']['yaw']}" />
   </joint>
   <joint name="os_lidar_fr_joint" type="fixed">
-    <parent link="rs16" />
+    <parent link="sensor_top" />
     <child link="os_lidar_fr" />
     <origin
-      xyz="${calibration['rs16']['os_lidar_fr']['x']}
-            ${calibration['rs16']['os_lidar_fr']['y']}
-            ${calibration['rs16']['os_lidar_fr']['z']}"
-      rpy="${calibration['rs16']['os_lidar_fr']['roll']}
-            ${calibration['rs16']['os_lidar_fr']['pitch']}
-            ${calibration['rs16']['os_lidar_fr']['yaw']}" />
+      xyz="${calibration['sensor_top']['os_lidar_fr']['x']}
+            ${calibration['sensor_top']['os_lidar_fr']['y']}
+            ${calibration['sensor_top']['os_lidar_fr']['z']}"
+      rpy="${calibration['sensor_top']['os_lidar_fr']['roll']}
+            ${calibration['sensor_top']['os_lidar_fr']['pitch']}
+            ${calibration['sensor_top']['os_lidar_fr']['yaw']}" />
   </joint>
    <joint name="os_lidar_rl_joint" type="fixed">
-    <parent link="rs16" />
+    <parent link="sensor_top" />
     <child link="os_lidar_rl" />
     <origin
-      xyz="${calibration['rs16']['os_lidar_rl']['x']}
-            ${calibration['rs16']['os_lidar_rl']['y']}
-            ${calibration['rs16']['os_lidar_rl']['z']}"
-      rpy="${calibration['rs16']['os_lidar_rl']['roll']}
-            ${calibration['rs16']['os_lidar_rl']['pitch']}
-            ${calibration['rs16']['os_lidar_rl']['yaw']}" />
+      xyz="${calibration['sensor_top']['os_lidar_rl']['x']}
+            ${calibration['sensor_top']['os_lidar_rl']['y']}
+            ${calibration['sensor_top']['os_lidar_rl']['z']}"
+      rpy="${calibration['sensor_top']['os_lidar_rl']['roll']}
+            ${calibration['sensor_top']['os_lidar_rl']['pitch']}
+            ${calibration['sensor_top']['os_lidar_rl']['yaw']}" />
   </joint>
    <joint name="os_lidar_rr_joint" type="fixed">
-    <parent link="rs16" />
+    <parent link="sensor_top" />
     <child link="os_lidar_rr" />
     <origin
-      xyz="${calibration['rs16']['os_lidar_rr']['x']}
-            ${calibration['rs16']['os_lidar_rr']['y']}
-            ${calibration['rs16']['os_lidar_rr']['z']}"
-      rpy="${calibration['rs16']['os_lidar_rr']['roll']}
-            ${calibration['rs16']['os_lidar_rr']['pitch']}
-            ${calibration['rs16']['os_lidar_rr']['yaw']}" />
+      xyz="${calibration['sensor_top']['os_lidar_rr']['x']}
+            ${calibration['sensor_top']['os_lidar_rr']['y']}
+            ${calibration['sensor_top']['os_lidar_rr']['z']}"
+      rpy="${calibration['sensor_top']['os_lidar_rr']['roll']}
+            ${calibration['sensor_top']['os_lidar_rr']['pitch']}
+            ${calibration['sensor_top']['os_lidar_rr']['yaw']}" />
   </joint>
 <!-- combined navigation -->
   <joint name="gnss_joint" type="fixed">
-    <parent link="rs16" />
+    <parent link="sensor_top" />
     <child link="gnss" />
     <origin
-      xyz="${calibration['rs16']['gnss']['x']}
-            ${calibration['rs16']['gnss']['y']}
-            ${calibration['rs16']['gnss']['z']}"
-      rpy="${calibration['rs16']['gnss']['roll']}
-            ${calibration['rs16']['gnss']['pitch']}
-            ${calibration['rs16']['gnss']['yaw']}" />
+      xyz="${calibration['sensor_top']['gnss']['x']}
+            ${calibration['sensor_top']['gnss']['y']}
+            ${calibration['sensor_top']['gnss']['z']}"
+      rpy="${calibration['sensor_top']['gnss']['roll']}
+            ${calibration['sensor_top']['gnss']['pitch']}
+            ${calibration['sensor_top']['gnss']['yaw']}" />
   </joint>
 </robot>

File: robobus_sensor_kit_description/urdf/sensors_secondary.xacro (robot description, xacro)
@@ -4,5 +4,5 @@
   <xacro:property name="secondary_calibration" value="${xacro.load_yaml('$(arg config_dir)/sensors_secondary_calibration.yaml')}"/>
   <!-- sensor secondary link -->
-  <link name="rs16" />
+  <link name="sensor_top" />
   <link name="front_radar" />
   <link name="rear_radar" />
@@ -21,14 +21,14 @@
   <!-- sensor kit joint -->
   <!-- lidar -->
-  <joint name="rs16_joint" type="fixed">
+  <joint name="sensor_top_joint" type="fixed">
     <parent link="base_link" />
-    <child link="rs16" />
+    <child link="sensor_top" />
     <origin
-      xyz="${secondary_calibration['base_link']['rs16']['x']}
-            ${secondary_calibration['base_link']['rs16']['y']}
-            ${secondary_calibration['base_link']['rs16']['z']}"
-      rpy="${secondary_calibration['base_link']['rs16']['roll']}
-            ${secondary_calibration['base_link']['rs16']['pitch']}
-            ${secondary_calibration['base_link']['rs16']['yaw']}" />
+      xyz="${secondary_calibration['base_link']['sensor_top']['x']}
+            ${secondary_calibration['base_link']['sensor_top']['y']}
+            ${secondary_calibration['base_link']['sensor_top']['z']}"
+      rpy="${secondary_calibration['base_link']['sensor_top']['roll']}
+            ${secondary_calibration['base_link']['sensor_top']['pitch']}
+            ${secondary_calibration['base_link']['sensor_top']['yaw']}" />
   </joint>
   <!-- millimeter wave -->
